Commit message: Gazebo

File: src/lidar_bot_unal/urdf/my_bot.urdf.xacro (robot description, xacro)
@@ -1,14 +1,22 @@
 <?xml version="1.0"?>
 <robot xmlns:xacro="http://www.ros.org/wiki/xacro" name="my_bot">
-  <!-- Parámetros globales -->
-  <xacro:property name="wheel_radius" value="0.05"/>
-  <xacro:property name="wheel_width"  value="0.02"/>
-  <xacro:property name="base_length"  value="0.30"/>
-  <xacro:property name="base_width"   value="0.30"/>
-  <xacro:property name="base_height"  value="0.08"/>
-  <!-- Material simple -->
+  <!-- =========================================================
+       PARÁMETROS GENERALES
+       ========================================================= -->
+  <xacro:property name="wheel_radius"     value="0.05"/>   <!-- 5 cm -->
+  <xacro:property name="wheel_width"      value="0.02"/>
+  <xacro:property name="base_length"      value="0.30"/>
+  <xacro:property name="base_width"       value="0.30"/>
+  <xacro:property name="base_height"      value="0.08"/>
+  <xacro:property name="wheel_separation" value="${base_width}"/>
+  <xacro:property name="wheel_diam"       value="${2*wheel_radius}"/>
+  <!-- =========================================================
+       MATERIALES
+       ========================================================= -->
   <material name="chassis_color"><color rgba="0.1 0.1 0.1 1"/></material>
   <material name="wheel_color"><color rgba="0.15 0.15 0.15 1"/></material>
-  <!-- Chasis -->
+  <!-- =========================================================
+       CHASIS
+       ========================================================= -->
   <link name="base_link">
     <visual>
@@ -28,11 +36,10 @@
       <mass value="4.0"/>
       <origin xyz="0 0 ${base_height/2}" rpy="0 0 0"/>
-      <inertia
-        ixx="0.02" ixy="0.0" ixz="0.0"
-        iyy="0.03" iyz="0.0"
-        izz="0.04"/>
+      <inertia ixx="0.02" ixy="0.0" ixz="0.0" iyy="0.03" iyz="0.0" izz="0.04"/>
     </inertial>
   </link>
-  <!-- Ruedas: izquierda y derecha -->
+  <!-- =========================================================
+       MACRO RUEDA
+       ========================================================= -->
   <xacro:macro name="wheel" params="side sign">
     <link name="${side}_wheel_link">
@@ -53,8 +60,6 @@
         <mass value="0.5"/>
         <origin xyz="0 0 0" rpy="0 0 0"/>
-        <inertia
-          ixx="0.0005" ixy="0.0" ixz="0.0"
-          iyy="0.0005" iyz="0.0"
-          izz="0.001"/>
+        <inertia ixx="0.0005" ixy="0.0" ixz="0.0"
+                 iyy="0.0005" iyz="0.0" izz="0.001"/>
       </inertial>
     </link>
@@ -66,8 +71,10 @@
     </joint>
   </xacro:macro>
-  <!-- Instanciación -->
+  <!-- Instanciación de ruedas -->
   <xacro:wheel side="left"  sign=" 1"/>
   <xacro:wheel side="right" sign="-1"/>
-  <!-- Sensor LIDAR (Hokuyo) -->
+  <!-- =========================================================
+       SENSOR LIDAR
+       ========================================================= -->
   <link name="laser_link">
     <visual>
@@ -84,3 +91,50 @@
     <origin xyz="0 0 ${base_height+0.05}" rpy="0 0 0"/>
   </joint>
+  <!-- =========================================================
+       PLUGINS GAZEBO
+       ========================================================= -->
+  <!-- Dif-Drive                                               -->
+  <gazebo>
+    <plugin name="diff_drive" filename="libgazebo_ros_diff_drive.so">
+      <left_joint>left_wheel_joint</left_joint>
+      <right_joint>right_wheel_joint</right_joint>
+      <wheel_separation>${wheel_separation}</wheel_separation>
+      <wheel_diameter>${wheel_diam}</wheel_diameter>
+      <publish_odom>true</publish_odom>
+      <odom_frame>odom</odom_frame>
+      <robot_base_frame>base_link</robot_base_frame>
+      <cmd_vel_topic>cmd_vel</cmd_vel_topic>
+      <odometry_topic>odom</odometry_topic>
+      <update_rate>50</update_rate>
+    </plugin>
+  </gazebo>
+  <!-- LIDAR como sensor ray   -->
+  <gazebo reference="laser_link">
+    <sensor type="ray" name="lidar">
+      <update_rate>20</update_rate>
+      <ray>
+        <scan>
+          <horizontal>
+            <samples>720</samples>
+            <resolution>1</resolution>
+            <min_angle>-1.5708</min_angle>
+            <max_angle>1.5708</max_angle>
+          </horizontal>
+        </scan>
+        <range>
+          <min>0.12</min>
+          <max>6.0</max>
+        </range>
+      </ray>
+      <plugin name="gazebo_laser" filename="libgazebo_ros_ray_sensor.so">
+        <ros>
+          <!-- remapea la salida interna ~/out a /scan -->
+          <remapping>~/out:=scan</remapping>
+        </ros>
+        <!-- publica LaserScan en vez de PointCloud2 -->
+        <output_type>sensor_msgs/LaserScan</output_type>
+        <frame_name>laser_link</frame_name>
+      </plugin>
+    </sensor>
+  </gazebo>
 </robot>

Commit message: Model Changes

File: src/lidar_bot_unal/urdf/my_bot.urdf.xacro (robot description, xacro)
@@ -6,7 +6,7 @@
   <xacro:property name="wheel_radius"     value="0.05"/>   <!-- 5 cm -->
   <xacro:property name="wheel_width"      value="0.02"/>
-  <xacro:property name="base_length"      value="0.30"/>
+  <xacro:property name="base_length"      value="0.25"/>
   <xacro:property name="base_width"       value="0.30"/>
-  <xacro:property name="base_height"      value="0.08"/>
+  <xacro:property name="base_height"      value="0.06"/>
   <xacro:property name="wheel_separation" value="${base_width}"/>
   <xacro:property name="wheel_diam"       value="${2*wheel_radius}"/>
@@ -14,6 +14,7 @@
        MATERIALES
        ========================================================= -->
-  <material name="chassis_color"><color rgba="0.1 0.1 0.1 1"/></material>
-  <material name="wheel_color"><color rgba="0.15 0.15 0.15 1"/></material>
+  <material name="chassis_color"><color rgba="0.3 0.5 0.8 1"/></material>
+  <material name="lidar_color"><color rgba="1.0 0.5 0.5 1"/></material>
+  <material name="wheel_color"><color rgba="0.6 0.6 0.6 1"/></material>
   <!-- =========================================================
        CHASIS
@@ -24,5 +25,5 @@
         <box size="${base_length} ${base_width} ${base_height}"/>
       </geometry>
-      <origin xyz="0 0 ${base_height/2}" rpy="0 0 0"/>
+      <origin xyz="0 0 ${wheel_radius}" rpy="0 0 0"/>
       <material name="chassis_color"/>
     </visual>
@@ -31,9 +32,9 @@
         <box size="${base_length} ${base_width} ${base_height}"/>
       </geometry>
-      <origin xyz="0 0 ${base_height/2}" rpy="0 0 0"/>
+      <origin xyz="0 0 ${wheel_radius}" rpy="0 0 0"/>
     </collision>
     <inertial>
       <mass value="4.0"/>
-      <origin xyz="0 0 ${base_height/2}" rpy="0 0 0"/>
+      <origin xyz="0 0 ${wheel_radius}" rpy="0 0 0"/>
       <inertia ixx="0.02" ixy="0.0" ixz="0.0" iyy="0.03" iyz="0.0" izz="0.04"/>
     </inertial>
@@ -82,6 +83,6 @@
         <cylinder length="0.02" radius="0.04"/>
       </geometry>
-      <origin xyz="0 0 ${base_height+0.05}" rpy="0 0 0"/>
-      <material name="chassis_color"/>
+      <origin xyz="0 0 ${base_height}" rpy="0 0 0"/>
+      <material name="lidar_color"/>
     </visual>
   </link>
@@ -89,5 +90,5 @@
     <parent link="base_link"/>
     <child  link="laser_link"/>
-    <origin xyz="0 0 ${base_height+0.05}" rpy="0 0 0"/>
+    <origin xyz="0 0 ${base_height}" rpy="0 0 0"/>
   </joint>
   <!-- =========================================================

Commit message: Initial navigation

File: src/lidar_bot_unal/urdf/my_bot.urdf.xacro (robot description, xacro)
@@ -90,5 +90,5 @@
     <parent link="base_link"/>
     <child  link="laser_link"/>
-    <origin xyz="0 0 ${base_height}" rpy="0 0 0"/>
+    <origin xyz="${base_length/2 + 0.01} 0 ${base_height}" rpy="0 0 0"/>
   </joint>
   <!-- =========================================================

Commit message: Model chasis visual

File: src/lidar_bot_unal/urdf/my_bot.urdf.xacro (robot description, xacro)
@@ -21,4 +21,5 @@
        ========================================================= -->
   <link name="base_link">
+    <!-- Visual for the main body -->
     <visual>
       <geometry>
@@ -28,4 +29,13 @@
       <material name="chassis_color"/>
     </visual>
+    <!-- Visual for the LiDAR support bracket (COSMETIC ONLY) -->
+    <visual name="lidar_support_visual">
+      <geometry>
+        <box size="0.035 0.05 0.09"/>
+      </geometry>
+      <origin xyz="${base_length/2} 0 ${base_height + 0.02}" rpy="0 0 0"/>
+      <material name="chassis_color"/>
+    </visual>
+    <!-- Collision for the main body (Unchanged) -->
     <collision>
       <geometry>
@@ -34,4 +44,5 @@
       <origin xyz="0 0 ${wheel_radius}" rpy="0 0 0"/>
     </collision>
+    <!-- Inertial properties (Unchanged) -->
     <inertial>
       <mass value="4.0"/>

Commit message: Añadidas paredes delimitadoras al mundo simulado y actualizado el diseño del robot para incluir cuatro ruedas, mejorando su estabilidad

File: src/lidar_bot_unal/urdf/my_bot.urdf.xacro (robot description, xacro)
@@ -24,7 +24,7 @@
     <visual>
       <geometry>
-        <box size="${base_length} ${base_width} ${base_height}"/>
+        <box size="${base_length} ${base_width} ${base_height}" rpy="0 0 0"/>
       </geometry>
-      <origin xyz="0 0 ${wheel_radius}" rpy="0 0 0"/>
+      <origin xyz="0 0 ${wheel_radius + base_height/2}"/>
       <material name="chassis_color"/>
     </visual>
@@ -42,5 +42,5 @@
         <box size="${base_length} ${base_width} ${base_height}"/>
       </geometry>
-      <origin xyz="0 0 ${wheel_radius}" rpy="0 0 0"/>
+      <origin xyz="0 0 ${wheel_radius + base_height/2}"/>
     </collision>
     <!-- Inertial properties (Unchanged) -->
@@ -54,36 +54,40 @@
        MACRO RUEDA
        ========================================================= -->
-  <xacro:macro name="wheel" params="side sign">
-    <link name="${side}_wheel_link">
-      <visual>
-        <geometry>
-          <cylinder length="${wheel_width}" radius="${wheel_radius}"/>
-        </geometry>
-        <origin xyz="0 0 0" rpy="1.5708 0 0"/>
-        <material name="wheel_color"/>
-      </visual>
-      <collision>
-        <geometry>
-          <cylinder length="${wheel_width}" radius="${wheel_radius}"/>
-        </geometry>
-        <origin xyz="0 0 0" rpy="1.5708 0 0"/>
-      </collision>
-      <inertial>
-        <mass value="0.5"/>
-        <origin xyz="0 0 0" rpy="0 0 0"/>
-        <inertia ixx="0.0005" ixy="0.0" ixz="0.0"
-                 iyy="0.0005" iyz="0.0" izz="0.001"/>
-      </inertial>
-    </link>
-    <joint name="${side}_wheel_joint" type="continuous">
-      <parent link="base_link"/>
-      <child  link="${side}_wheel_link"/>
-      <origin xyz="0 ${sign*base_width/2} ${wheel_radius}" rpy="0 0 0"/>
-      <axis xyz="0 1 0"/>
-    </joint>
-  </xacro:macro>
+  <xacro:macro name="wheel" params="name x_offset y_offset">
+  <link name="${name}_link">
+    <visual>
+      <geometry>
+        <cylinder length="${wheel_width}" radius="${wheel_radius}"/>
+      </geometry>
+      <origin xyz="0 0 0" rpy="1.5708 0 0"/>
+      <material name="wheel_color"/>
+    </visual>
+    <collision>
+      <geometry>
+        <cylinder length="${wheel_width}" radius="${wheel_radius}"/>
+      </geometry>
+      <origin xyz="0 0 0" rpy="1.5708 0 0"/>
+    </collision>
+    <inertial>
+      <mass value="0.5"/>
+      <origin xyz="0 0 0" rpy="0 0 0"/>
+      <inertia ixx="0.0005" ixy="0.0" ixz="0.0"
+               iyy="0.0005" iyz="0.0" izz="0.001"/>
+    </inertial>
+  </link>
+  <joint name="${name}_joint" type="continuous">
+    <parent link="base_link"/>
+    <child  link="${name}_link"/>
+    <origin xyz="${x_offset} ${y_offset} ${wheel_radius}" rpy="0 0 0"/>
+    <axis xyz="0 1 0"/>
+  </joint>
+</xacro:macro>
   <!-- Instanciación de ruedas -->
-  <xacro:wheel side="left"  sign=" 1"/>
-  <xacro:wheel side="right" sign="-1"/>
+  <!-- Ruedas delanteras -->
+<xacro:wheel name="front_left_wheel"  x_offset="${ base_length/2 - 0.05}" y_offset=" ${ base_width/2}" />
+<xacro:wheel name="front_right_wheel" x_offset="${ base_length/2 - 0.05}" y_offset="-${ base_width/2}" />
+<!-- Ruedas traseras -->
+<xacro:wheel name="rear_left_wheel"   x_offset="-${ base_length/2 - 0.05}" y_offset=" ${ base_width/2}" />
+<xacro:wheel name="rear_right_wheel"  x_offset="-${ base_length/2 - 0.05}" y_offset="-${ base_width/2}" />
   <!-- =========================================================
        SENSOR LIDAR
@@ -109,6 +113,6 @@
   <gazebo>
     <plugin name="diff_drive" filename="libgazebo_ros_diff_drive.so">
-      <left_joint>left_wheel_joint</left_joint>
-      <right_joint>right_wheel_joint</right_joint>
+      <left_joint>rear_left_wheel_joint</left_joint>
+      <right_joint>rear_right_wheel_joint</right_joint>
       <wheel_separation>${wheel_separation}</wheel_separation>
       <wheel_diameter>${wheel_diam}</wheel_diameter>
